File: versions/v0.9.2/hardware/KiCad_files/PCB layout/Shield v0.9.2/Shield_v0.9.2.kicad_pcb (KiCad board)
At the start: 2 copper layers, 71.5 x 50.2 mm, 34 parts, among them J1 Conn_01x15, J2 Conn_01x15, P1 CONN_01X02, P3 CONN_01X10, P4 CONN_01X01, P5 CONN_01X01, U1 EL3H7, U2 FDC1004custom

Commit message: Added Logos
Parts:
- added G***: LOGO, LOGO, B.Cu at (155.5, 70.5)
- added G***: LOGO, LOGO, B.Cu at (137.5, 70.5)
Other:
- board text added: "9/9/2026"
- board text added: "Mani Asadi"
- board text added: "SEC-DAQ"
- board text added: "v0.9.2"
