File: versions/v0.9.2/hardware/KiCad_files/PCB layout/Shield v0.9.2/Shield_v0.9.2.kicad_sch (KiCad schematic)
At the start: 32 parts, among them J1 Conn_01x15, J2 Conn_01x15, P1 CONN_01X02, P3 CONN_01X10, P4 CONN_01X01, P5 CONN_01X01, U1 EL3H7, U2 FDC1004custom

Commit message: Added Logos
Other:
- note added: "V0.9.2"
- note removed: "V0.3"
Changed lines of the file:
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@@
 		)
 	)
-	(text "V0.3"
+	(text "V0.9.2"
 		(exclude_from_sim no)
 		(at 190.5 180.34 0)
@@
 		)
 		(instances
-			(project "Shield_V0.3"
+			(project "Shield_v0.9.2"
 				(path "/5b3a0963-f29a-46c5-9178-369cd6a02136"
 					(reference "P1")
@@
 		)
 		(instances
-			(project "Shield_V0.3"
+			(project "Shield_v0.9.2"
 				(path "/5b3a0963-f29a-46c5-9178-369cd6a02136"
 					(reference "R1")
@@
 		)
 		(instances
-			(project "Shield_V0.3"
+			(project "Shield_v0.9.2"
 				(path "/5b3a0963-f29a-46c5-9178-369cd6a02136"
 					(reference "#PWR18")
@@
 		)
 		(instances
-			(project "Shield_V0.3"
+			(project "Shield_v0.9.2"
 				(path "/5b3a0963-f29a-46c5-9178-369cd6a02136"
 					(reference "R2")
@@
 		)
 		(instances
-			(project "Shield_V0.3"
+			(project "Shield_v0.9.2"
 				(path "/5b3a0963-f29a-46c5-9178-369cd6a02136"
 					(reference "#PWR16")
@@
 		)
 		(instances
-			(project "Shield_V0.3"
+			(project "Shield_v0.9.2"
 				(path "/5b3a0963-f29a-46c5-9178-369cd6a02136"
 					(reference "S_Range1")
@@
 		)
 		(instances
-			(project "Shield_V0.3"
+			(project "Shield_v0.9.2"
 				(path "/5b3a0963-f29a-46c5-9178-369cd6a02136"
 					(reference "R7")
@@
 		)
 		(instances
-			(project "Shield_V0.3"
+			(project "Shield_v0.9.2"
 				(path "/5b3a0963-f29a-46c5-9178-369cd6a02136"
 					(reference "R8")
@@
 		)
 		(instances
-			(project "Shield_V0.3"
+			(project "Shield_v0.9.2"
 				(path "/5b3a0963-f29a-46c5-9178-369cd6a02136"
 					(reference "#PWR5")
@@
 		)
 		(instances
-			(project "Shield_V0.3"
+			(project "Shield_v0.9.2"
 				(path "/5b3a0963-f29a-46c5-9178-369cd6a02136"
 					(reference "S_Channel1")
@@
 		)
 		(instances
-			(project "Shield_V0.3"
+			(project "Shield_v0.9.2"
 				(path "/5b3a0963-f29a-46c5-9178-369cd6a02136"
 					(reference "S_Sample1")
@@
 		)
 		(instances
-			(project "Shield_V0.3"
+			(project "Shield_v0.9.2"
 				(path "/5b3a0963-f29a-46c5-9178-369cd6a02136"
 					(reference "R6")
@@
 		)
 		(instances
-			(project "Shield_V0.3"
+			(project "Shield_v0.9.2"
 				(path "/5b3a0963-f29a-46c5-9178-369cd6a02136"
 					(reference "R5")
@@
 		)
 		(instances
-			(project "Shield_V0.3"
+			(project "Shield_v0.9.2"
 				(path "/5b3a0963-f29a-46c5-9178-369cd6a02136"
 					(reference "R4")
@@
 		)
 		(instances
-			(project "Shield_V0.3"
+			(project "Shield_v0.9.2"
 				(path "/5b3a0963-f29a-46c5-9178-369cd6a02136"
 					(reference "R3")
@@
 		)
 		(instances
-			(project "Shield_V0.3"
+			(project "Shield_v0.9.2"
 				(path "/5b3a0963-f29a-46c5-9178-369cd6a02136"
 					(reference "#PWR6")
@@
 		)
 		(instances
-			(project "Shield_V0.3"
+			(project "Shield_v0.9.2"
 				(path "/5b3a0963-f29a-46c5-9178-369cd6a02136"
 					(reference "#PWR3")
@@
 		)
 		(instances
-			(project "Shield_V0.3"
+			(project "Shield_v0.9.2"
 				(path "/5b3a0963-f29a-46c5-9178-369cd6a02136"
 					(reference "#PWR2")
@@
 		)
 		(instances
-			(project "Shield_V0.3"
+			(project "Shield_v0.9.2"
 				(path "/5b3a0963-f29a-46c5-9178-369cd6a02136"
 					(reference "#PWR4")
@@
 		)
 		(instances
-			(project "Shield_V0.3"
+			(project "Shield_v0.9.2"
 				(path "/5b3a0963-f29a-46c5-9178-369cd6a02136"
 					(reference "S_Ground1")
@@
 		)
 		(instances
-			(project "Shield_V0.3"
+			(project "Shield_v0.9.2"
 				(path "/5b3a0963-f29a-46c5-9178-369cd6a02136"
 					(reference "S_Trigger1")
@@
 		)
 		(instances
-			(project "Shield_V0.3"
+			(project "Shield_v0.9.2"
 				(path "/5b3a0963-f29a-46c5-9178-369cd6a02136"
 					(reference "P3")
@@
 		)
 		(instances
-			(project "Shield_V0.3"
+			(project "Shield_v0.9.2"
 				(path "/5b3a0963-f29a-46c5-9178-369cd6a02136"
 					(reference "#PWR15")
@@
 		)
 		(instances
-			(project "Shield_V0.3"
+			(project "Shield_v0.9.2"
 				(path "/5b3a0963-f29a-46c5-9178-369cd6a02136"
 					(reference "U2")
@@
 		)
 		(instances
-			(project "Shield_V0.3"
+			(project "Shield_v0.9.2"
 				(path "/5b3a0963-f29a-46c5-9178-369cd6a02136"
 					(reference "#PWR11")
@@
 		)
 		(instances
-			(project "Shield_V0.3"
+			(project "Shield_v0.9.2"
 				(path "/5b3a0963-f29a-46c5-9178-369cd6a02136"
 					(reference "#PWR10")
@@
 		)
 		(instances
-			(project "Shield_V0.3"
+			(project "Shield_v0.9.2"
 				(path "/5b3a0963-f29a-46c5-9178-369cd6a02136"
 					(reference "RI2C1")
@@
 		)
 		(instances
-			(project "Shield_V0.3"
+			(project "Shield_v0.9.2"
 				(path "/5b3a0963-f29a-46c5-9178-369cd6a02136"
 					(reference "RI2C2")
@@
 		)
 		(instances
-			(project "Shield_V0.3"
+			(project "Shield_v0.9.2"
 				(path "/5b3a0963-f29a-46c5-9178-369cd6a02136"
 					(reference "#PWR12")
@@
 		)
 		(instances
-			(project "Shield_V0.3"
+			(project "Shield_v0.9.2"
 				(path "/5b3a0963-f29a-46c5-9178-369cd6a02136"
 					(reference "#PWR14")
@@
 		)
 		(instances
-			(project "Shield_V0.3"
+			(project "Shield_v0.9.2"
 				(path "/5b3a0963-f29a-46c5-9178-369cd6a02136"
 					(reference "#PWR19")
@@
 		)
 		(instances
-			(project "Shield_V0.3"
+			(project "Shield_v0.9.2"
 				(path "/5b3a0963-f29a-46c5-9178-369cd6a02136"
 					(reference "L1")
@@
 		)
 		(instances
-			(project "Shield_V0.3"
+			(project "Shield_v0.9.2"
 				(path "/5b3a0963-f29a-46c5-9178-369cd6a02136"
 					(reference "C3")
@@
 		)
 		(instances
-			(project "Shield_V0.3"
+			(project "Shield_v0.9.2"
 				(path "/5b3a0963-f29a-46c5-9178-369cd6a02136"
 					(reference "C5")
@@
 		)
 		(instances
-			(project "Shield_V0.3"
+			(project "Shield_v0.9.2"
 				(path "/5b3a0963-f29a-46c5-9178-369cd6a02136"
 					(reference "C6")
@@
 		)
 		(instances
-			(project "Shield_V0.3"
+			(project "Shield_v0.9.2"
 				(path "/5b3a0963-f29a-46c5-9178-369cd6a02136"
 					(reference "C7")
@@
 		)
 		(instances
-			(project "Shield_V0.3"
+			(project "Shield_v0.9.2"
 				(path "/5b3a0963-f29a-46c5-9178-369cd6a02136"
 					(reference "#PWR17")
@@
 		)
 		(instances
-			(project "Shield_V0.3"
+			(project "Shield_v0.9.2"
 				(path "/5b3a0963-f29a-46c5-9178-369cd6a02136"
 					(reference "P5")
@@
 		)
 		(instances
-			(project "Shield_V0.3"
+			(project "Shield_v0.9.2"
 				(path "/5b3a0963-f29a-46c5-9178-369cd6a02136"
 					(reference "P4")
@@
 		)
 		(instances
-			(project "Shield_V0.3"
+			(project "Shield_v0.9.2"
 				(path "/5b3a0963-f29a-46c5-9178-369cd6a02136"
 					(reference "#PWR1")
@@
 		)
 		(instances
-			(project "Shield_V0.3"
+			(project "Shield_v0.9.2"
 				(path "/5b3a0963-f29a-46c5-9178-369cd6a02136"
 					(reference "C1")
@@
 		)
 		(instances
-			(project "Shield_V0.3"
+			(project "Shield_v0.9.2"
 				(path "/5b3a0963-f29a-46c5-9178-369cd6a02136"
 					(reference "C2")
@@
 		)
 		(instances
-			(project "Shield_V0.3"
+			(project "Shield_v0.9.2"
 				(path "/5b3a0963-f29a-46c5-9178-369cd6a02136"
 					(reference "C4")
@@
 		)
 		(instances
-			(project "Shield_V0.3"
+			(project "Shield_v0.9.2"
 				(path "/5b3a0963-f29a-46c5-9178-369cd6a02136"
 					(reference "#PWR13")
@@
 		)
 		(instances
-			(project "Shield_V0.3"
+			(project "Shield_v0.9.2"
 				(path "/5b3a0963-f29a-46c5-9178-369cd6a02136"
 					(reference "U1")
@@
 		)
 		(instances
-			(project "Shield_V0.3"
+			(project "Shield_v0.9.2"
 				(path "/5b3a0963-f29a-46c5-9178-369cd6a02136"
 					(reference "#PWR9")
@@
 		)
 		(instances
-			(project "Shield_V0.3"
+			(project "Shield_v0.9.2"
 				(path "/5b3a0963-f29a-46c5-9178-369cd6a02136"
 					(reference "#FLG3")
@@
 		)
 		(instances
-			(project "Shield_V0.3"
+			(project "Shield_v0.9.2"
 				(path "/5b3a0963-f29a-46c5-9178-369cd6a02136"
 					(reference "#FLG2")
@@
 		)
 		(instances
-			(project "Shield_V0.3"
+			(project "Shield_v0.9.2"
 				(path "/5b3a0963-f29a-46c5-9178-369cd6a02136"
 					(reference "#FLG1")
@@
 		)
 		(instances
-			(project "Shield_V0.3"
+			(project "Shield_v0.9.2"
 				(path "/5b3a0963-f29a-46c5-9178-369cd6a02136"
 					(reference "#PWR7")
@@
 		)
 		(instances
-			(project "Shield_V0.3"
+			(project "Shield_v0.9.2"
 				(path "/5b3a0963-f29a-46c5-9178-369cd6a02136"
 					(reference "#PWR8")
@@
 		)
 		(instances
-			(project "Shield_V0.3"
+			(project "Shield_v0.9.2"
 				(path "/5b3a0963-f29a-46c5-9178-369cd6a02136"
 					(reference "GND1")
@@
 		)
 		(instances
-			(project "Shield_V0.3"
+			(project "Shield_v0.9.2"
 				(path "/5b3a0963-f29a-46c5-9178-369cd6a02136"
 					(reference "J1")
@@
 		)
 		(instances
-			(project "Shield_V0.3"
+			(project "Shield_v0.9.2"
 				(path "/5b3a0963-f29a-46c5-9178-369cd6a02136"
 					(reference "J2")
